File: enoki/hardware/enoki.kicad_pcb (KiCad board)
At the start: 2 copper layers, 102.9 x 57.1 mm, 48 parts, among them U1 ALLWINNERA10/TFBGA441, U2 H5TQ4G63MFR, U3 H5TQ4G63MFR, X1 32768Hz/6pF, X2 4SB24.000F20E15/5x3.2mm/20ppm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

Commit message: working on pcb
Parts:
- added C43, C44, C45, C46, C47, C48, C49, C50, C51, C52, C53, C54, C55, C57, C60, C61, C66, C67, C68, C69, C71, C72, C73, C75, C76, C77, C78, C79, C80, C81, C82, C83, C84, C85, C86, C87, C88, C89, C90, C91, C92, C93, C94, C95, C96, C97: 220nF, SMD_Packages:SM0402_c, F.Cu at (140.3, 143.4)
- added C56: 22uF/6.3v, SMD_Packages:SM0603_Capa, F.Cu at (140.3, 143.4)
- added C58, C59: 33pF, SMD_Packages:SM0402_c, F.Cu at (140.3, 143.4)
- added C62, C63: 10pF, SMD_Packages:SM0402_c, F.Cu at (140.3, 143.4)
- added C64, C70, C74: 22uF/6.3V, SMD_Packages:SM0603_Capa, F.Cu at (140.3, 143.4)
- added C65: 100nF, SMD_Packages:SM0402_c, F.Cu at (140.3, 143.4)
- added R10, R12, R6, R7, R9: 2K, SMD_Packages:SM0402_r, F.Cu at (140.3, 143.4)
- added R11, R4, R5: 330R, SMD_Packages:SM0402_r, F.Cu at (140.3, 143.4)
- added R13: 10M, SMD_Packages:SM0402_r, F.Cu at (140.3, 143.4)
- added R2: 22R, SMD_Packages:SM0402_r, F.Cu at (140.3, 143.4)
- added R3: 0R, SMD_Packages:SM0402_r, F.Cu at (140.3, 143.4)
- added R8: NA, SMD_Packages:SM0402_r, F.Cu at (140.3, 143.4)
- C1: value 220nF -> NA
- C15: value 220nF -> 22uF/6.3V
- C20: value 22uF/6.3v -> 220nF
- C33, C34: value 33pF -> 220nF
- C35: value 10pF -> 22OnF
- C36: value 10pF -> 220nF
- C37, C39, C41: value 22uF/6.3V -> 220nF
- C38: value 100nF -> 220nF
- R1: value 10M -> 22R
- X1: value 32768Hz/6pF -> 4SB24.000F20E15/5x3.2mm/20ppm/20pF
- X2: value 4SB24.000F20E15/5x3.2mm/20ppm/20pF -> 32768Hz/6pF
- moved U1 59.3 mm to (108.3, 94.0), turned to 180 degrees
- moved X1 34.3 mm to (188.0, 94.0), turned to 270 degrees
- moved X2 30.1 mm to (153.7, 80.0), turned to 180 degrees
- moved C35 26.7 mm to (166.4, 111.8)
- moved U3 13.3 mm to (131.1, 99.4), turned to 90 degrees
- moved U2 11.4 mm to (131.1, 88.0), turned to 90 degrees
- moved C24 7.73 mm to (166.4, 92.7)
- moved C27 7.62 mm to (166.4, 96.5)
- moved C16 4.02 mm to (166.4, 94.0)
Connections:
- C1 pad 1: Net-(C1-Pad1) -> GND
- C1 pad 2: GND -> CPU-REF
- C10 pad 1: +1.2V -> +1.5V
- C11 pad 1: +1.2V -> +1.5V
- C12 pad 1: +1.2V -> +1.2V_INT
- C13 pad 1: +1.2V -> +1.2V_INT
- C14 pad 1: +1.2V -> +1.2V_INT
- C15 pad 1: +1.2V -> +1.2V_INT
- C16 pad 1: Net-(C16-Pad1) -> +1.5V
- C17 pad 1: +3.3V -> +1.5V
- C18 pad 1: +3.3V -> +1.5V
- C19 pad 1: +3.3V -> +1.5V
- C2 pad 1: +1.2V -> +1.5V
- C20 pad 1: +3.3V -> +1.5V
- C21 pad 1: +3.3V -> +1.5V
- C22 pad 1: +3.3V -> +1.5V
- C23 pad 1: +3.3V -> +1.5V
- C24 pad 1: +3.3V -> +1.5V
- C25 pad 1: +3.3V -> +1.5V
- C26 pad 1: +3.3V -> +1.5V
- C27 pad 1: +3.3V -> +1.5V
- C28 pad 1: +3.3V -> +1.5V
- C29 pad 1: +3.3V -> +1.5V
- C3 pad 1: +1.2V -> +1.5V
- C30 pad 1: +3.3V -> +1.5V
- C31 pad 1: +3.3V -> +1.5V
- C32 pad 1: +3.3V -> +1.5V
- C33 pad 1: GND -> +1.5V
- C33 pad 2: Net-(C33-Pad2) -> GND
- C34 pad 1: GND -> +1.5V
- C34 pad 2: Net-(C34-Pad2) -> DDR_VREF
- C35 pad 1: GND -> DDR_VREF
- C35 pad 2: Net-(C35-Pad2) -> GND
- C36 pad 1: GND -> +1.5V
- C36 pad 2: Net-(C36-Pad2) -> GND
- C37 pad 1: GND -> +1.5V
- C37 pad 2: Net-(C37-Pad2) -> GND
- C38 pad 1: GND -> +1.5V
- C38 pad 2: Net-(C37-Pad2) -> GND
- C39 pad 1: +2.5V -> +1.5V
- C4 pad 1: +1.2V -> +1.5V
- C40 pad 1: +2.5V -> +1.5V
- C41 pad 1: +1.2V -> +1.5V
- C42 pad 1: +1.2V -> +1.5V
- C5 pad 1: +1.2V -> +1.5V
- C6 pad 1: +1.2V -> +1.5V
- C7 pad 1: +1.2V -> +1.5V
- C8 pad 1: +1.2V -> +1.5V
- C9 pad 1: +1.2V -> +1.5V
- R1 pad 1: Net-(C35-Pad2) -> /Sheet54FC94AD/CLK
- R1 pad 2: Net-(C36-Pad2) -> Net-(R1-Pad2)
- U1 pad AA1: Net-(U1-PadAA1) -> /Sheet54FC94AD/DQ12
- U1 pad AA2: Net-(U1-PadAA2) -> /Sheet54FC94AD/SDQS1_N
- U1 pad AA3: Net-(U1-PadAA3) -> /Sheet54FC94AD/SA8
- U1 pad AA8: Net-(U1-PadAA8) -> CPU-REF
- U1 pad AB1: Net-(U1-PadAB1) -> /Sheet54FC94AD/SDQM1
- U1 pad AB2: Net-(U1-PadAB2) -> /Sheet54FC94AD/DQ8
- U1 pad AB3: Net-(U1-PadAB3) -> /Sheet54FC94AD/DQ13
- U1 pad AB4: Net-(U1-PadAB4) -> /Sheet54FC94AD/DQ0
- U1 pad AB5: Net-(U1-PadAB5) -> /Sheet54FC94AD/DQ5
- U1 pad AB6: Net-(U1-PadAB6) -> /Sheet54FC94AD/SDQS0
- U1 pad AB7: Net-(U1-PadAB7) -> /Sheet54FC94AD/DQ6
- U1 pad AB8: Net-(U1-PadAB8) -> /Sheet54FC94AD/DQ3
- U1 pad AC1: Net-(U1-PadAC1) -> /Sheet54FC94AD/DQ15
- U1 pad AC2: Net-(U1-PadAC2) -> /Sheet54FC94AD/DQ10
- U1 pad AC3: (no net) -> /Sheet54FC94AD/DQ7
- U1 pad AC4: Net-(U1-PadAC4) -> /Sheet54FC94AD/DQ2
- U1 pad AC5: Net-(U1-PadAC5) -> /Sheet54FC94AD/SDQS0_N
- U1 pad AC6: Net-(U1-PadAC6) -> /Sheet54FC94AD/SDQM0
- U1 pad AC7: Net-(U1-PadAC7) -> /Sheet54FC94AD/DQ1
- U1 pad AC8: Net-(U1-PadAC8) -> /Sheet54FC94AD/DQ4
- U1 pad F1: Net-(C35-Pad2) -> Net-(C62-Pad2)
- U1 pad F2: Net-(C36-Pad2) -> Net-(C63-Pad2)
- U1 pad G1: Net-(U1-PadG1) -> /Sheet54FC94AD/SDQM3
- U1 pad G2: Net-(U1-PadG2) -> /Sheet54FC94AD/DQ30
- U1 pad G3: Net-(U1-PadG3) -> GND
- U1 pad G4: Net-(U1-PadG4) -> GND
- U1 pad G5: Net-(U1-PadG5) -> +1.5V
- U1 pad H1: Net-(U1-PadH1) -> /Sheet54FC94AD/DQ25
- U1 pad H2: Net-(U1-PadH2) -> /Sheet54FC94AD/DQ27
- U1 pad H3: Net-(U1-PadH3) -> CPU-REF
- U1 pad H4: Net-(U1-PadH4) -> CPU-REF
- U1 pad H5: Net-(U1-PadH5) -> +1.5V
- U1 pad J1: Net-(U1-PadJ1) -> /Sheet54FC94AD/DQ28
- U1 pad J2: Net-(U1-PadJ2) -> /Sheet54FC94AD/SDQS3_N
- U1 pad J5: Net-(U1-PadJ5) -> GND
- U1 pad K1: Net-(U1-PadK1) -> /Sheet54FC94AD/SDQS3
- U1 pad K2: Net-(U1-PadK2) -> /Sheet54FC94AD/DQ31
- U1 pad K3: Net-(U1-PadK3) -> /Sheet54FC94AD/BA0
- U1 pad K4: Net-(U1-PadK4) -> /Sheet54FC94AD/BA2
- U1 pad K5: Net-(U1-PadK5) -> GND
- U1 pad K8: Net-(C37-Pad2) -> Net-(C64-Pad2)
- U1 pad L1: Net-(U1-PadL1) -> /Sheet54FC94AD/DQ24
- U1 pad L2: Net-(U1-PadL2) -> /Sheet54FC94AD/DQ26
- U1 pad L3: Net-(U1-PadL3) -> /Sheet54FC94AD/SA10
- U1 pad L4: Net-(U1-PadL4) -> /Sheet54FC94AD/BA1
- U1 pad L5: Net-(U1-PadL5) -> +1.5V
- U1 pad L8: Net-(C16-Pad1) -> Net-(C97-Pad1)
- U1 pad M1: Net-(U1-PadM1) -> /Sheet54FC94AD/DQ29
- U1 pad M13: GND -> Net-(U1-PadM13)
- U1 pad M2: Net-(U1-PadM2) -> /Sheet54FC94AD/DQ23
- U1 pad M3: Net-(U1-PadM3) -> /Sheet54FC94AD/SA7
- U1 pad M4: Net-(U1-PadM4) -> /Sheet54FC94AD/SA3
- U1 pad M5: Net-(U1-PadM5) -> +1.5V
- U1 pad M8: Net-(U1-PadM8) -> +1.2V_INT
- U1 pad M9: Net-(U1-PadM9) -> GND
- U1 pad N1: Net-(U1-PadN1) -> /Sheet54FC94AD/DQ16
- U1 pad N10: Net-(U1-PadN10) -> GND
- U1 pad N2: Net-(U1-PadN2) -> /Sheet54FC94AD/DQ18
- U1 pad N22: Net-(C34-Pad2) -> Net-(C59-Pad2)
- U1 pad N23: Net-(C33-Pad2) -> Net-(C58-Pad2)
- U1 pad N3: Net-(U1-PadN3) -> /Sheet54FC94AD/CKE
- U1 pad N4: Net-(U1-PadN4) -> /Sheet54FC94AD/SA5
- U1 pad N5: Net-(U1-PadN5) -> GND
- U1 pad N9: Net-(U1-PadN9) -> +1.2V_INT
- U1 pad P1: Net-(U1-PadP1) -> /Sheet54FC94AD/DQ21
- U1 pad P10: Net-(U1-PadP10) -> GND
- U1 pad P2: Net-(U1-PadP2) -> /Sheet54FC94AD/SDQS2_N
- U1 pad P3: Net-(U1-PadP3) -> /Sheet54FC94AD/SA12
- U1 pad P4: Net-(U1-PadP4) -> /Sheet54FC94AD/SA9
- U1 pad P5: Net-(U1-PadP5) -> GND
- U1 pad P9: Net-(U1-PadP9) -> +1.2V_INT
- U1 pad R1: Net-(U1-PadR1) -> /Sheet54FC94AD/SDQS2
- U1 pad R11: GND -> Net-(U1-PadF19)
- U1 pad R2: Net-(U1-PadR2) -> /Sheet54FC94AD/SDQM2
- U1 pad R3: Net-(U1-PadR3) -> /Sheet54FC94AD/SA14
- U1 pad R4: Net-(U1-PadR4) -> /Sheet54FC94AD/SA1
- U1 pad R5: Net-(U1-PadR5) -> +1.5V
- U1 pad T1: Net-(U1-PadT1) -> /Sheet54FC94AD/DQ22
- U1 pad T2: Net-(U1-PadT2) -> /Sheet54FC94AD/DQ17
- U1 pad T3: Net-(U1-PadT3) -> /Sheet54FC94AD/WEN
- U1 pad T4: Net-(U1-PadT4) -> /Sheet54FC94AD/RASN
- U1 pad T5: Net-(U1-PadT5) -> +1.5V
- U1 pad U1: Net-(U1-PadU1) -> /Sheet54FC94AD/DQ19
- U1 pad U2: Net-(U1-PadU2) -> /Sheet54FC94AD/DQ20
- U1 pad U3: Net-(U1-PadU3) -> /Sheet54FC94AD/CASN
- U1 pad U4: Net-(U1-PadU4) -> /Sheet54FC94AD/SA2
- U1 pad U5: Net-(U1-PadU5) -> GND
- U1 pad V1: Net-(U1-PadV1) -> Net-(R1-Pad2)
- U1 pad V4: Net-(U1-PadV4) -> /Sheet54FC94AD/SA6
- U1 pad V5: Net-(U1-PadV5) -> GND
- U1 pad W1: Net-(U1-PadW1) -> /Sheet54FC94AD/SDQM1
- U1 pad W2: Net-(U1-PadW2) -> /Sheet54FC94AD/DQ14
- U1 pad W3: Net-(U1-PadW3) -> /Sheet54FC94AD/SA11
- U1 pad W4: Net-(U1-PadW4) -> /Sheet54FC94AD/SA0
- U1 pad W5: Net-(U1-PadW5) -> +1.5V
- U1 pad W6: Net-(U1-PadW6) -> +1.5V
- U1 pad W7: Net-(U1-PadW7) -> +1.5V
- U1 pad Y1: Net-(U1-PadY1) -> /Sheet54FC94AD/DQ9
- U1 pad Y2: Net-(U1-PadY2) -> /Sheet54FC94AD/DQ11
- U1 pad Y3: Net-(U1-PadY3) -> /Sheet54FC94AD/SA13
- U1 pad Y4: Net-(U1-PadY4) -> /Sheet54FC94AD/SA4
- U1 pad Y5: Net-(U1-PadY5) -> CPU-REF
- U1 pad Y6: Net-(U1-PadY6) -> +1.5V
- U1 pad Y7: Net-(U1-PadY7) -> GND
- U1 pad Y8: Net-(U1-PadY8) -> GND
- U2 pad A1: (no net) -> +1.5V
- U2 pad A2: (no net) -> /Sheet54FC94AD/DQ13
- U2 pad A3: (no net) -> /Sheet54FC94AD/DQ15
- U2 pad A7: (no net) -> /Sheet54FC94AD/DQ12
- U2 pad A8: (no net) -> +1.5V
- U2 pad A9: (no net) -> GND
- U2 pad B1: (no net) -> GND
- U2 pad B2: (no net) -> +1.5V
- U2 pad B3: (no net) -> GND
- U2 pad B7: (no net) -> /Sheet54FC94AD/SDQS1_N
- U2 pad B8: (no net) -> /Sheet54FC94AD/DQ14
- U2 pad B9: (no net) -> +1.5V
- U2 pad C1: (no net) -> +1.5V
- U2 pad C2: (no net) -> /Sheet54FC94AD/DQ11
- U2 pad C3: (no net) -> /Sheet54FC94AD/DQ9
- U2 pad C7: (no net) -> /Sheet54FC94AD/SDQS1
- U2 pad C8: (no net) -> /Sheet54FC94AD/DQ10
- U2 pad C9: (no net) -> +1.5V
- U2 pad D1: (no net) -> GND
- U2 pad D2: (no net) -> +1.5V
- U2 pad D3: (no net) -> /Sheet54FC94AD/SDQM1
- U2 pad D7: (no net) -> /Sheet54FC94AD/DQ8
- U2 pad D8: (no net) -> GND
- U2 pad E1: (no net) -> GND
- U2 pad E2: (no net) -> GND
- U2 pad E3: (no net) -> /Sheet54FC94AD/DQ0
- U2 pad E7: (no net) -> /Sheet54FC94AD/SDQM0
- U2 pad E8: (no net) -> GND
- U2 pad E9: (no net) -> +1.5V
- U2 pad F1: (no net) -> +1.5V
- U2 pad F2: (no net) -> /Sheet54FC94AD/DQ2
- U2 pad F3: (no net) -> /Sheet54FC94AD/SDQS0
- U2 pad F7: (no net) -> /Sheet54FC94AD/DQ1
- U2 pad F8: (no net) -> /Sheet54FC94AD/DQ3
- U2 pad F9: (no net) -> GND
- U2 pad G1: (no net) -> GND
- U2 pad G2: (no net) -> /Sheet54FC94AD/DQ6
- U2 pad G3: (no net) -> /Sheet54FC94AD/SDQS0_N
- U2 pad G7: (no net) -> +1.5V
- U2 pad G8: (no net) -> GND
- U2 pad G9: (no net) -> GND
- U2 pad H1: (no net) -> DDR_VREF
- U2 pad H2: (no net) -> +1.5V
- U2 pad H3: (no net) -> /Sheet54FC94AD/DQ4
- U2 pad H7: (no net) -> /Sheet54FC94AD/DQ7
- U2 pad H8: (no net) -> /Sheet54FC94AD/DQ5
- U2 pad H9: (no net) -> +1.5V
- U2 pad J1: (no net) -> Net-(U2-PadJ1)
- U2 pad J2: (no net) -> GND
- U2 pad J3: (no net) -> /Sheet54FC94AD/RASN
- U2 pad J7: (no net) -> /Sheet54FC94AD/CLK
- U2 pad J8: (no net) -> GND
- U2 pad J9: (no net) -> Net-(U2-PadJ9)
- U2 pad K1: (no net) -> /Sheet54FC94AD/DDR3_ODT
- U2 pad K2: (no net) -> +1.5V
- U2 pad K3: (no net) -> /Sheet54FC94AD/CASN
- U2 pad K7: (no net) -> /Sheet54FC94AD/CLKN
- U2 pad K8: (no net) -> +1.5V
- U2 pad K9: (no net) -> /Sheet54FC94AD/CKE
- U2 pad L1: (no net) -> Net-(U2-PadL1)
- U2 pad L2: (no net) -> /Sheet54FC94AD/SCS0
- U2 pad L3: (no net) -> /Sheet54FC94AD/WEN
- U2 pad L7: (no net) -> /Sheet54FC94AD/SA10
- U2 pad L8: (no net) -> Net-(R5-Pad2)
- U2 pad L9: (no net) -> Net-(U2-PadL9)
- U2 pad M1: (no net) -> GND
- U2 pad M2: (no net) -> /Sheet54FC94AD/BA0
- U2 pad M3: (no net) -> /Sheet54FC94AD/BA2
- U2 pad M7: (no net) -> Net-(U2-PadM7)
- U2 pad M8: (no net) -> DDR_VREF
- U2 pad M9: (no net) -> GND
- U2 pad N1: (no net) -> +1.5V
- U2 pad N2: (no net) -> /Sheet54FC94AD/SA3
- U2 pad N3: Net-(U2-PadN3) -> /Sheet54FC94AD/SA0
- U2 pad N7: (no net) -> /Sheet54FC94AD/SA12
- U2 pad N8: (no net) -> /Sheet54FC94AD/BA1
- U2 pad N9: (no net) -> +1.5V
- U2 pad P1: (no net) -> GND
- U2 pad P2: (no net) -> /Sheet54FC94AD/SA5
- U2 pad P3: (no net) -> /Sheet54FC94AD/SA2
- U2 pad P7: (no net) -> /Sheet54FC94AD/SA1
- U2 pad P8: (no net) -> /Sheet54FC94AD/SA4
- U2 pad P9: (no net) -> GND
- U2 pad R1: (no net) -> +1.5V
- U2 pad R2: (no net) -> /Sheet54FC94AD/SA7
- U2 pad R3: (no net) -> /Sheet54FC94AD/SA9
- U2 pad R7: (no net) -> /Sheet54FC94AD/SA11
- U2 pad R8: (no net) -> /Sheet54FC94AD/SA6
- U2 pad R9: (no net) -> +1.5V
- U2 pad T1: (no net) -> GND
- U2 pad T2: (no net) -> /Sheet54FC94AD/DDR3_RST
- U2 pad T3: (no net) -> /Sheet54FC94AD/SA13
- U2 pad T7: (no net) -> /Sheet54FC94AD/SA14
- U2 pad T8: (no net) -> /Sheet54FC94AD/SA8
- U2 pad T9: (no net) -> GND
- U3 pad A1: (no net) -> +1.5V
- U3 pad A2: (no net) -> /Sheet54FC94AD/DQ29
- U3 pad A3: (no net) -> /Sheet54FC94AD/DQ31
- U3 pad A7: (no net) -> /Sheet54FC94AD/DQ28
- U3 pad A8: (no net) -> +1.5V
- U3 pad A9: (no net) -> GND
- U3 pad B1: (no net) -> GND
- U3 pad B2: (no net) -> +1.5V
- U3 pad B3: (no net) -> GND
- U3 pad B7: (no net) -> /Sheet54FC94AD/SDQS3_N
- U3 pad B8: (no net) -> /Sheet54FC94AD/DQ30
- U3 pad B9: (no net) -> +1.5V
- U3 pad C1: (no net) -> +1.5V
- U3 pad C2: (no net) -> /Sheet54FC94AD/DQ27
- U3 pad C3: (no net) -> /Sheet54FC94AD/DQ25
- U3 pad C7: (no net) -> /Sheet54FC94AD/SDQS3
- U3 pad C8: (no net) -> /Sheet54FC94AD/DQ26
- U3 pad C9: (no net) -> +1.5V
- U3 pad D1: (no net) -> GND
- U3 pad D2: (no net) -> +1.5V
- U3 pad D3: (no net) -> /Sheet54FC94AD/SDQM3
- U3 pad D7: (no net) -> /Sheet54FC94AD/DQ24
- U3 pad D8: (no net) -> GND
- U3 pad E1: (no net) -> GND
- U3 pad E2: (no net) -> GND
- U3 pad E3: (no net) -> /Sheet54FC94AD/DQ16
- U3 pad E7: (no net) -> /Sheet54FC94AD/SDQM2
- U3 pad E8: (no net) -> GND
- U3 pad E9: (no net) -> +1.5V
- U3 pad F1: (no net) -> +1.5V
- U3 pad F2: (no net) -> /Sheet54FC94AD/DQ18
- U3 pad F3: (no net) -> /Sheet54FC94AD/SDQS2
- U3 pad F7: (no net) -> /Sheet54FC94AD/DQ17
- U3 pad F8: (no net) -> /Sheet54FC94AD/DQ19
- U3 pad F9: (no net) -> GND
- U3 pad G1: (no net) -> GND
- U3 pad G2: (no net) -> /Sheet54FC94AD/DQ22
- U3 pad G3: (no net) -> /Sheet54FC94AD/SDQS2_N
- U3 pad G7: (no net) -> +1.5V
- U3 pad G8: (no net) -> GND
- U3 pad G9: (no net) -> GND
- U3 pad H1: (no net) -> DDR_VREF
- U3 pad H2: (no net) -> +1.5V
- U3 pad H3: (no net) -> /Sheet54FC94AD/DQ20
- U3 pad H7: (no net) -> /Sheet54FC94AD/DQ23
- U3 pad H8: (no net) -> /Sheet54FC94AD/DQ21
- U3 pad H9: (no net) -> +1.5V
- U3 pad J1: (no net) -> Net-(U3-PadJ1)
- U3 pad J2: (no net) -> GND
- U3 pad J3: (no net) -> /Sheet54FC94AD/RASN
- U3 pad J7: (no net) -> /Sheet54FC94AD/CLK
- U3 pad J8: (no net) -> GND
- U3 pad J9: (no net) -> Net-(U3-PadJ9)
- U3 pad K1: (no net) -> /Sheet54FC94AD/DDR3_ODT
- U3 pad K2: (no net) -> +1.5V
- U3 pad K3: (no net) -> /Sheet54FC94AD/CASN
- U3 pad K7: (no net) -> /Sheet54FC94AD/CLKN
- U3 pad K8: (no net) -> +1.5V
- U3 pad K9: (no net) -> /Sheet54FC94AD/CKE
- U3 pad L1: (no net) -> Net-(U3-PadL1)
- U3 pad L2: (no net) -> /Sheet54FC94AD/SCS0
- U3 pad L3: (no net) -> /Sheet54FC94AD/WEN
- U3 pad L7: (no net) -> /Sheet54FC94AD/SA10
- U3 pad L8: (no net) -> Net-(R11-Pad2)
- U3 pad L9: (no net) -> Net-(U3-PadL9)
- U3 pad M1: (no net) -> GND
- U3 pad M2: (no net) -> /Sheet54FC94AD/BA0
- U3 pad M3: (no net) -> /Sheet54FC94AD/BA2
- U3 pad M7: (no net) -> Net-(U3-PadM7)
- U3 pad M8: (no net) -> DDR_VREF
- U3 pad M9: (no net) -> GND
- U3 pad N1: (no net) -> +1.5V
- U3 pad N2: (no net) -> /Sheet54FC94AD/SA3
- U3 pad N3: Net-(U3-PadN3) -> /Sheet54FC94AD/SA0
- U3 pad N7: (no net) -> /Sheet54FC94AD/SA12
- U3 pad N8: (no net) -> /Sheet54FC94AD/BA1
- U3 pad N9: (no net) -> +1.5V
- U3 pad P1: (no net) -> GND
- U3 pad P2: (no net) -> /Sheet54FC94AD/SA5
- U3 pad P3: (no net) -> /Sheet54FC94AD/SA2
- U3 pad P7: (no net) -> /Sheet54FC94AD/SA1
- U3 pad P8: (no net) -> /Sheet54FC94AD/SA4
- U3 pad P9: (no net) -> GND
- U3 pad R1: (no net) -> +1.5V
- U3 pad R2: (no net) -> /Sheet54FC94AD/SA7
- U3 pad R3: (no net) -> /Sheet54FC94AD/SA9
- U3 pad R7: (no net) -> /Sheet54FC94AD/SA11
- U3 pad R8: (no net) -> /Sheet54FC94AD/SA6
- U3 pad R9: (no net) -> +1.5V
- U3 pad T1: (no net) -> GND
- U3 pad T2: (no net) -> /Sheet54FC94AD/DDR3_RST
- U3 pad T3: (no net) -> /Sheet54FC94AD/SA13
- U3 pad T7: (no net) -> /Sheet54FC94AD/SA14
- U3 pad T8: (no net) -> /Sheet54FC94AD/SA8
- U3 pad T9: (no net) -> GND
- X1 pad 1: Net-(C36-Pad2) -> Net-(C59-Pad2)
- X1 pad 2: Net-(C35-Pad2) -> Net-(C58-Pad2)
- X2 pad 1: Net-(C34-Pad2) -> Net-(C63-Pad2)
- X2 pad 2: Net-(C33-Pad2) -> Net-(C62-Pad2)
Routing:
- net /Sheet54FC94AD/DQ0: track 0.00 -> 15.1 mm, vias 0 -> 2
- net /Sheet54FC94AD/SDQM1: track 0.00 -> 12.0 mm, vias 0 -> 2
- net /Sheet54FC94AD/DQ13: track 0.00 -> 11.7 mm
- net /Sheet54FC94AD/DQ11: track 0.00 -> 11.5 mm, vias 0 -> 2
- net /Sheet54FC94AD/DQ9: track 0.00 -> 10.6 mm, vias 0 -> 2
- net /Sheet54FC94AD/DQ15: track 0.00 -> 9.77 mm
- net (no net): track 0.00 -> 6.01 mm
- net /Sheet54FC94AD/DQ26: track 0.00 -> 0.68 mm
- net +1.2V: track 0.00 -> 0.61 mm
Other:
- copper layers 2 -> 4
- net class Default: clearance 0.254 -> 0.09144; trace_width 0.254 -> 0.1524; via_dia 0.889 -> 0.4572; via_drill 0.635 -> 0.2032
- net class power added: clearance 0.09144, trace_width 0.1524, via_dia 0.4572, via_drill 0.2032
- rule trace_clearance: 0.254 -> 0.09144
- rule trace_min: 0.254 -> 0.127
- rule via_min_drill: 0.508 -> 0.2032
- rule via_min_size: 0.889 -> 0.4064
