File: enoki/hardware/file54FC94AD.sch (KiCad schematic (older format))
At the start: 3 parts, among them U1 ALLWINNERA10/TFBGA441, U2 H5TQ4G63MFR, U3 H5TQ4G63MFR

Commit message: ram lib ok
Connections:
- net DQU7: now reaches U2.A3 (DQU7)
Other:
- moved on the sheet: U2, U3
Changed lines of the file:
@@
 	1    0    0    -1
 $EndComp
-Wire Bus Line
-	10500 900  10500 6500
-Wire Bus Line
-	6350 5650 6350 4100
-Wire Bus Line
-	6350 4100 10500 4100
-Entry Wire Line
-	6250 4200 6350 4300
-Entry Wire Line
-	6250 4300 6350 4400
-Entry Wire Line
-	6250 4400 6350 4500
-Entry Wire Line
-	6250 4500 6350 4600
-Entry Wire Line
-	6250 4600 6350 4700
-Entry Wire Line
-	6250 4700 6350 4800
-Entry Wire Line
-	6250 4800 6350 4900
-Entry Wire Line
-	6250 4900 6350 5000
-Entry Wire Line
-	6250 5000 6350 5100
-Entry Wire Line
-	6250 5100 6350 5200
-Entry Wire Line
-	6250 5200 6350 5300
-Entry Wire Line
-	6250 5300 6350 5400
-Entry Wire Line
-	6250 5400 6350 5500
-Entry Wire Line
-	6250 5500 6350 5600
-Entry Wire Line
-	6250 5600 6350 5700
-Wire Bus Line
-	6350 5700 6350 5600
-Wire Bus Line
-	1550 6000 1550 900
-Wire Bus Line
-	1150 900  10500 900
-Entry Wire Line
-	1550 2400 1650 2500
-Entry Wire Line
-	1550 2500 1650 2600
-Entry Wire Line
-	1550 2600 1650 2700
-Entry Wire Line
-	1550 2800 1650 2900
-Entry Wire Line
-	1550 2900 1650 3000
-Entry Wire Line
-	1550 3000 1650 3100
-Entry Wire Line
-	1550 3100 1650 3200
-Entry Wire Line
-	1550 3300 1650 3400
-Entry Wire Line
-	1550 3200 1650 3300
-Entry Wire Line
-	1550 3400 1650 3500
-Entry Wire Line
-	1550 3500 1650 3600
-Entry Wire Line
-	1550 3600 1650 3700
-Entry Wire Line
-	1550 3700 1650 3800
-Entry Wire Line
-	1550 3800 1650 3900
-Entry Wire Line
-	1550 3900 1650 4000
-Entry Wire Line
-	1550 4000 1650 4100
-Entry Wire Line
-	1550 4100 1650 4200
-Entry Wire Line
-	1550 4200 1650 4300
-Entry Wire Line
-	1550 4300 1650 4400
-Entry Wire Line
-	1550 4400 1650 4500
-Entry Wire Line
-	1550 4500 1650 4600
-Entry Wire Line
-	1550 4600 1650 4700
-Entry Wire Line
-	1550 4700 1650 4800
-Entry Wire Line
-	1550 4800 1650 4900
-Entry Wire Line
-	1550 4900 1650 5000
-Entry Wire Line
-	1550 5000 1650 5100
-Entry Wire Line
-	1550 5100 1650 5200
-Entry Wire Line
-	1550 5200 1650 5300
-Entry Wire Line
-	1550 5300 1650 5400
-Entry Wire Line
-	1550 5400 1650 5500
-Entry Wire Line
-	1550 5500 1650 5600
-Entry Wire Line
-	1550 5600 1650 5700
-Entry Wire Line
-	1550 5700 1650 5800
-Entry Wire Line
-	1550 5800 1650 5900
-Entry Wire Line
-	1550 5900 1650 6000
 $Comp
 L H5TQ4G63MFR U2
 U 1 1 54FF604E
-P 13900 3750
-F 0 "U2" H 13900 3750 60  0000 C CNN
-F 1 "H5TQ4G63MFR" H 13900 3750 60  0000 C CNN
-F 2 "" H 13900 3750 60  0000 C CNN
-F 3 "" H 13900 3750 60  0000 C CNN
-	1    13900 3750
+P 14450 3900
+F 0 "U2" H 14450 3900 60  0000 C CNN
+F 1 "H5TQ4G63MFR" H 14450 3900 60  0000 C CNN
+F 2 "" H 14450 3900 60  0000 C CNN
+F 3 "" H 14450 3900 60  0000 C CNN
+	1    14450 3900
 	1    0    0    -1
 $EndComp
@@
 L H5TQ4G63MFR U3
 U 1 1 54FF6062
-P 22250 3800
-F 0 "U3" H 22250 3800 60  0000 C CNN
-F 1 "H5TQ4G63MFR" H 22250 3800 60  0000 C CNN
-F 2 "" H 22250 3800 60  0000 C CNN
-F 3 "" H 22250 3800 60  0000 C CNN
-	1    22250 3800
+P 21950 4000
+F 0 "U3" H 21950 4000 60  0000 C CNN
+F 1 "H5TQ4G63MFR" H 21950 4000 60  0000 C CNN
+F 2 "" H 21950 4000 60  0000 C CNN
+F 3 "" H 21950 4000 60  0000 C CNN
+	1    21950 4000
 	1    0    0    -1
 $EndComp
+Wire Bus Line
+	1050 6900 1050 750
+Wire Bus Line
+	16050 750  16050 3500
+Entry Wire Line
+	15950 1850 16050 1950
+Entry Wire Line
+	15950 1950 16050 2050
+Entry Wire Line
+	15950 2050 16050 2150
+Entry Wire Line
+	15950 2150 16050 2250
+Entry Wire Line
+	15950 2250 16050 2350
+Entry Wire Line
+	15950 2350 16050 2450
+Entry Wire Line
+	15950 2550 16050 2650
+Entry Wire Line
+	15950 2450 16050 2550
+Wire Bus Line
+	1050 750  16050 750
+Wire Wire Line
+	15950 1850 15650 1850
+Wire Wire Line
+	15650 1950 15950 1950
+Wire Wire Line
+	15650 2050 15950 2050
+Wire Wire Line
+	15950 2150 15650 2150
+Wire Wire Line
+	15650 2250 15950 2250
+Wire Wire Line
+	15950 2350 15650 2350
+Wire Wire Line
+	15650 2450 15950 2450
+Wire Wire Line
+	15950 2550 15650 2550
+Text Label 15700 1850 0    60   ~ 0
+DQU7
 $EndSCHEMATC

Commit message: working on pcb
Parts:
- added C1: NA, symbol C
- added C10, C11, C12, C13, C14, C16, C17, C18, C19, C2, C20, C21, C22, C23, C24, C25, C26, C27, C28, C29, C3, C30, C31, C32, C33, C34, C36, C37, C38, C39, C4, C40, C41, C42, C43, C44, C45, C46, C47, C48, C49, C5, C50, C51, C52, C53, C54, C55, C6, C7, C8, C9: 220nF, symbol C
- added C15: 22uF/6.3V, symbol C
- added C35: 22OnF, symbol C
- added R1, R2: 22R, symbol R
- added R10, R12, R6, R7, R9: 2K, symbol R
- added R11, R4, R5: 330R, symbol R
- added R3: 0R, symbol R
- added R8: NA, symbol R
Connections:
- net DQU7 is gone; now on net DQ15: U2.A3 (DQU7)
- net DQ12: now reaches U1.AA1 (SDQ12)
- net DQ12: now also U2.A7 (DQU4)
- net SDQS1_N: now reaches U1.AA2 (SDQS1#)
- net SDQS1_N: now also U2.B7 (#DQSU)
- net SA8: now reaches U1.AA3 (SA8)
- net SA8: now also U2.T8 (A8), U3.T8 (A8)
- net at U1.AA5 (SODT0): now also R3.2
- net at U1.AA7 (SZQ): now also R4.2
- net CPU-REF: now reaches U1.AA8 (SVREF3)
- net CPU-REF: now also U1.H3 (SVREF0), U1.H4 (SVREF1), U1.Y5 (SVREF2), C1.2, C46.2, C47.1, R10.1, R8.1, R9.2
- net SDQM1: now reaches U1.AB1 (SDQS1)
- net SDQM1: now also U1.W1 (SDQM1), U2.D3 (DMU)
- net DQ8: now reaches U1.AB2 (SDQ8)
- net DQ8: now also U2.D7 (DQU0)
- net DQ13: now reaches U1.AB3 (SDQ13)
- net DQ13: now also U2.A2 (DQU5)
- net DQ0: now reaches U1.AB4 (SDQ0)
- net DQ0: now also U2.E3 (DQL0)
- net DQ5: now reaches U1.AB5 (SDQ5)
- net DQ5: now also U2.H8 (DQL5)
- net SDQS0: now reaches U1.AB6 (SDQS0)
- net SDQS0: now also U2.F3 (DQSL)
- net DQ6: now reaches U1.AB7 (SDQ6)
- net DQ6: now also U2.G2 (DQL6)
- net DQ3: now reaches U1.AB8 (SDQ3)
- net DQ3: now also U2.F8 (DQL3)
- net DQ15: now reaches U1.AC1 (SDQ15)
- net DQ10: now reaches U1.AC2 (SDQ10)
- net DQ10: now also U2.C8 (DQU2)
- net DQ7: now reaches U1.AC3 (SDQ7)
- net DQ7: now also U2.H7 (DQL7)
- net DQ2: now reaches U1.AC4 (SDQ2)
- net DQ2: now also U2.F2 (DQL2)
- net SDQS0_N: now reaches U1.AC5 (SDQS0#)
- net SDQS0_N: now also U2.G3 (#DQSL)
- net SDQM0: now reaches U1.AC6 (SDQM0)
- net SDQM0: now also U2.E7 (DML)
- net DQ1: now reaches U1.AC7 (SDQ1)
- net DQ1: now also U2.F7 (DQL1)
- net DQ4: now reaches U1.AC8 (SDQ4)
- net DQ4: now also U2.H3 (DQL4)
- net SDQM3: now reaches U1.G1 (SDQM3)
- net SDQM3: now also U3.D3 (DMU)
- net DQ30: now reaches U1.G2 (SDQ30)
- net DQ30: now also U3.B8 (DQU6)
- net GND: now reaches U1.G3 (GND_DRAM)
- net GND: now also U1.G4 (GND_DRAM), U1.J5 (GND_DRAM), U1.K5 (GND_DRAM), U1.M9 (GND_DLL), U1.N10 (GND_DLL), U1.N5 (GND_DRAM), U1.P10 (GND_DLL), U1.P5 (GND_DRAM), U1.U5 (GND_DRAM), U1.V5 (GND_DRAM), U1.Y7 (GND_DRAM), U1.Y8 (GND_DRAM), U2.A9 (VSS), U2.B1 (VSSQ), U2.B3 (VSS), U2.B9 (VSSQ), U2.D1 (VSSQ), U2.D8 (VSSQ), U2.E1 (VSS), U2.E2 (VSSQ), U2.E8 (VSSQ), U2.F9 (VSSQ), U2.G1 (VSSQ), U2.G8 (VSS), U2.G9 (VSSQ), U2.J2 (VSS), U2.J8 (VSS), U2.M1 (VSS), U2.M9 (VSS), U2.P1 (VSS), U2.P9 (VSS), U2.T1 (VSS), U2.T9 (VSS), U3.A9 (VSS), U3.B1 (VSSQ), U3.B3 (VSS), U3.B9 (VSSQ), U3.D1 (VSSQ), U3.D8 (VSSQ), U3.E1 (VSS), U3.E2 (VSSQ), U3.E8 (VSSQ), U3.F9 (VSSQ), U3.G1 (VSSQ), U3.G8 (VSS), U3.G9 (VSSQ), U3.J2 (VSS), U3.J8 (VSS), U3.M1 (VSS), U3.M9 (VSS), U3.P1 (VSS), U3.P9 (VSS), U3.T1 (VSS), U3.T9 (VSS), C1.1, C10.2, C11.2, C12.2, C13.2, C14.2, C15.2, C16.2, C17.2, C18.2, C19.2, C2.2, C20.2, C21.2, C22.2, C23.2, C24.2, C25.2, C26.2, C27.2, C28.2, C29.2, C3.2, C30.2, C31.2, C32.2, C33.2, C35.2, C36.2, C37.2, C38.2, C39.2, C4.2, C40.2, C41.2, C42.2, C43.2, C44.2, C45.2, C47.2, C48.2, C49.2, C5.2, C50.2, C51.2, C52.2, C53.2, C54.2, C55.2, C6.2, C7.2, C8.2, C9.2, R10.2, R11.1, R4.1, R5.1, R7.2
- net +1.5V: now reaches U1.G5 (VCC_DRAM)
- net +1.5V: now also U1.H5 (VCC_DRAM), U1.L5 (VCC_DRAM), U1.M5 (VCC_DRAM), U1.R5 (VCC_DRAM), U1.T5 (VCC_DRAM), U1.W5 (VCC_DRAM), U1.W6 (VCC_DRAM), U1.W7 (VCC_DRAM), U1.Y6 (VCC_DRAM), U2.A1 (VDDQ), U2.A8 (VDDQ), U2.B2 (VDD), U2.B9 (VSSQ), U2.C1 (VDDQ), U2.C9 (VDDQ), U2.D2 (VDDQ), U2.E9 (VDDQ), U2.F1 (VDDQ), U2.G7 (VDD), U2.H2 (VDDQ), U2.H9 (VDDQ), U2.K2 (VDD), U2.K8 (VDD), U2.N1 (VDD), U2.N9 (VDD), U2.R1 (VDD), U2.R9 (VDD), U3.A1 (VDDQ), U3.A8 (VDDQ), U3.B2 (VDD), U3.B9 (VSSQ), U3.C1 (VDDQ), U3.C9 (VDDQ), U3.D2 (VDDQ), U3.E9 (VDDQ), U3.F1 (VDDQ), U3.G7 (VDD), U3.H2 (VDDQ), U3.H9 (VDDQ), U3.K2 (VDD), U3.K8 (VDD), U3.N1 (VDD), U3.N9 (VDD), U3.R1 (VDD), U3.R9 (VDD), C10.1, C11.1, C16.1, C17.1, C18.1, C19.1, C2.1, C20.1, C21.1, C22.1, C23.1, C24.1, C25.1, C26.1, C27.1, C28.1, C29.1, C3.1, C30.1, C31.1, C32.1, C33.1, C34.1, C36.1, C37.1, C38.1, C39.1, C4.1, C40.1, C41.1, C42.1, C43.1, C44.1, C45.1, C46.1, C48.1, C49.1, C5.1, C50.1, C51.1, C52.1, C53.1, C54.1, C55.1, C6.1, C7.1, C8.1, C9.1, R12.1, R6.1, R9.1
- net DQ25: now reaches U1.H1 (SDQ25)
- net DQ25: now also U3.C3 (DQU1)
- net DQ27: now reaches U1.H2 (SDQ27)
- net DQ27: now also U3.C2 (DQU3)
- net DQ28: now reaches U1.J1 (SDQ28)
- net DQ28: now also U3.A7 (DQU4)
- net SDQS3_N: now reaches U1.J2 (SDQS3#)
- net SDQS3_N: now also U3.B7 (#DQSU)
- net SDQS3: now reaches U1.K1 (SDQS3)
- net SDQS3: now also U3.C7 (DQSU)
- net DQ31: now reaches U1.K2 (SDQ31)
- net DQ31: now also U3.A3 (DQU7)
- net BA0: now reaches U1.K3 (SBA0)
- net BA0: now also U2.M2 (BA0), U3.M2 (BA0)
- net BA2: now reaches U1.K4 (SBA2)
- net BA2: now also U2.M3 (BA2), U3.M3 (BA2)
- net DQ24: now reaches U1.L1 (SDQ24)
- net DQ24: now also U3.D7 (DQU0)
- net DQ26: now reaches U1.L2 (SDQ26)
- net DQ26: now also U3.C8 (DQU2)
- net SA10: now reaches U1.L3 (SA10)
- net SA10: now also U2.L7 (A10/AP), U3.L7 (A10/AP)
- net BA1: now reaches U1.L4 (SBA1)
- net BA1: now also U2.N8 (BA1), U3.N8 (BA1)
- net DQ29: now reaches U1.M1 (SDQ29)
- net DQ29: now also U3.A2 (DQU5)
- net DQ23: now reaches U1.M2 (SDQ23)
- net DQ23: now also U3.H7 (DQL7)
- net SA7: now reaches U1.M3 (SA7)
- net SA7: now also U2.R2 (A7), U3.R2 (A7)
- net SA3: now reaches U1.M4 (SA3)
- net SA3: now also U2.N2 (A3), U3.N2 (A3)
- net +1.2V_INT: now reaches U1.M8 (VDD_DLL)
- net +1.2V_INT: now also U1.N9 (VDD_DLL), U1.P9 (VDD_DLL), C12.1, C13.1, C14.1, C15.1
- net DQ16: now reaches U1.N1 (SDQ16)
- net DQ16: now also U3.E3 (DQL0)
- net DQ18: now reaches U1.N2 (SDQ18)
- net DQ18: now also U3.F2 (DQL2)
- net CKE: now reaches U1.N3 (SCKE0)
- net CKE: now also U2.K9 (CKE), U3.K9 (CKE)
- net SA5: now reaches U1.N4 (SA5)
- net SA5: now also U2.P2 (A5), U3.P2 (A5)
- net DQ21: now reaches U1.P1 (SDQ21)
- net DQ21: now also U3.H8 (DQL5)
- net SDQS2_N: now reaches U1.P2 (SDQS2#)
- net SDQS2_N: now also U3.G3 (#DQSL)
- net SA12: now reaches U1.P3 (SA12)
- net SA12: now also U2.N7 (A12/#BC), U3.N7 (A12/#BC)
- net SA9: now reaches U1.P4 (SA9)
- net SA9: now also U2.R3 (A9), U3.R3 (A9)
- net SDQS2: now reaches U1.R1 (SDQS2)
- net SDQS2: now also U3.F3 (DQSL)
- net SDQM2: now reaches U1.R2 (SDQM2)
- net SDQM2: now also U3.E7 (DML)
- net SA14: now reaches U1.R3 (SA14)
- net SA14: now also U2.T7 (A14/NC), U3.T7 (A14/NC)
- net SA1: now reaches U1.R4 (SA1)
- net SA1: now also U2.P7 (A1), U3.P7 (A1)
- net DQ22: now reaches U1.T1 (SDQ22)
- net DQ22: now also U3.G2 (DQL6)
- net DQ17: now reaches U1.T2 (SDQ17)
- net DQ17: now also U3.F7 (DQL1)
- net WEN: now reaches U1.T3 (SWE)
- net WEN: now also U2.L3 (#WE), U3.L3 (#WE)
- net RASN: now reaches U1.T4 (SRAS)
- net RASN: now also U2.J3 (#RAS), U3.J3 (#RAS)
- net DQ19: now reaches U1.U1 (SDQ19)
- net DQ19: now also U3.F8 (DQL3)
- net DQ20: now reaches U1.U2 (SDQ20)
- net DQ20: now also U3.H3 (DQL4)
- net CASN: now reaches U1.U3 (SCAS)
- net CASN: now also U2.K3 (#CAS), U3.K3 (#CAS)
- net SA2: now reaches U1.U4 (SA2)
- net SA2: now also U2.P3 (A2), U3.P3 (A2)
- net at U1.V1 (SCK): now also R1.2
- net at U1.V2 (SCK#): now also R2.2
- net SA6: now reaches U1.V4 (SA6)
- net SA6: now also U2.R8 (A6), U3.R8 (A6)
- net DQ14: now reaches U1.W2 (SDQ14)
- net DQ14: now also U2.B8 (DQU6)
- net SA11: now reaches U1.W3 (SA11)
- net SA11: now also U2.R7 (A11), U3.R7 (A11)
- net SA0: now reaches U1.W4 (SA0)
- net SA0: now also U2.N3 (A0), U3.N3 (A0)
- net DQ9: now reaches U1.Y1 (SDQ9)
- net DQ9: now also U2.C3 (DQU1)
- net DQ11: now reaches U1.Y2 (SDQ11)
- net DQ11: now also U2.C2 (DQU3)
- net SA13: now reaches U1.Y3 (SA13)
- net SA13: now also U2.T3 (A13), U3.T3 (A13)
- net SA4: now reaches U1.Y4 (SA4)
- net SA4: now also U2.P8 (A4), U3.P8 (A4)
- net SDQS1: now reaches U2.C7 (DQSU)
- net DDR_VREF: now reaches U2.H1 (VREFDQ)
- net DDR_VREF: now also U2.M8 (VREFCA), U3.H1 (VREFDQ), U3.M8 (VREFCA), C34.2, C35.1, R6.2, R7.1, R8.2
- net CLK: now reaches U2.J7 (CK)
- net CLK: now also U3.J7 (CK), R1.1
- net DDR3_ODT: now reaches U2.K1 (ODT)
- net DDR3_ODT: now also U3.K1 (ODT), R3.1
- net CLKN: now reaches U2.K7 (#CK)
- net CLKN: now also U3.K7 (#CK), R2.1
- net SCS0: now reaches U2.L2 (#CS)
- net SCS0: now also U3.L2 (#CS)
- net at U2.L8 (ZQ): now also R5.2
- net DDR3_RST: now reaches U2.T2 (#RESET)
- net DDR3_RST: now also U3.T2 (#RESET), R12.2
- net at U3.L8 (ZQ): now also R11.2
- no-connect marks 0 -> 12
Other:
- note added: "DDR3 RAM"
- moved on the sheet: U1C, U2, U3
