File: enoki/hardware/powers.sch (KiCad schematic (older format))
At the start: 46 parts, among them U1 ALLWINNERA10/TFBGA441, X1 32768Hz/6pF, X2 4SB24.000F20E15/5x3.2mm/20ppm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

Commit message: working on pcb
Parts:
- renumbered C20 to C56, C21 to C57, C33 to C58, C34 to C59, C22 to C60, C23 to C61, C35 to C62, C36 to C63, C37 to C64, C38 to C65, C24 to C66, C25 to C67, C26 to C68, C27 to C69, C39 to C70, C28 to C71, C40 to C72, C29 to C73, C41 to C74, C30 to C75, C42 to C76, C31 to C77, C32 to C78, C1 to C79, C2 to C80, C3 to C81, C4 to C82, C17 to C83, C5 to C84, C18 to C85, C6 to C86, C19 to C87, C7 to C88, C8 to C89, C9 to C90, C10 to C91, C11 to C92, C12 to C93, C13 to C94, C14 to C95, C15 to C96, C16 to C97, R1 to R13, X2 to X1, X1 to X2
